File: RML/RML.kicad_sch (KiCad schematic)
At the start: 29 parts, among them Q101 Q_NMOS_GDS, Q102 Q_NMOS_GDS, U101 641964-1, U102 LM555xM, U103 SFH617A-1, U104 74AHC1G02, U105 641964-1, U106 641964-1, U107 LM7805_TO220

Commit message: Checked RML
Other:
- note added: "satisfied"
