File: RML/RML.kicad_pcb (KiCad board)
At the start: 4 copper layers, 85 x 50 mm, 29 parts, among them Q101 Q_NMOS_GDS, Q102 Q_NMOS_GDS, U101 641964-1, U102 LM555xM, U103 SFH617A-1, U104 74AHC1G02, U105 641964-1, U106 641964-1, U107 LM7805_TO220

Commit message: Checked RML
Parts:
- added G***: LOGO, LOGO, F.Cu at (119.2, 81.1)
- added G***: LOGO, LOGO, F.Cu at (111.0, 82.5)
- added G***: LOGO, LOGO, F.Cu at (117.5, 44.5)
Routing:
- net GND: vias 206 -> 165
Other:
- board text added: "4.5mm"
- board text added: "GROUNDED LOW VOLTAGE"
