File: RML/Through Hole Testing/RML.kicad_sch (KiCad schematic)
At the start: 29 parts, among them Q101 Q_NMOS_GDS, Q102 Q_NMOS_GDS, U101 641964-1, U102 LM555xM, U103 SFH617A-1, U104 74AHC1G02, U105 641964-1, U106 641964-1, U107 LM7805_TO220

Commit message: RML Through hole BOM updated
Parts:
- C101: Through Hole Digikey (none) -> https://www.digikey.com/en/products/detail/kemet/C330C105K5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; Through hole Manufacturing Part Number (none) -> K105K20X7RF5TH5
- C102: Through Hole Digikey (none) -> https://www.digikey.com/en/products/detail/vishay-beyschlag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; Through hole Manufacturing Part Number (none) -> K104K10X7RF5UH5
- C103, C106: Through Hole Digikey (none) -> https://www.digikey.com/en/products/detail/vishay-beyschlag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; Through hole Manufacturing Part Number (none) -> A103K15X7RF5TAA
- C104: Through Hole Digikey (none) -> https://www.digikey.com/en/products/detail/tdk-corporation/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; Through hole Manufacturing Part Number (none) -> FK14X5R0J226MR020
- C105: Through Hole Digikey (none) -> https://www.digikey.com/en/products/detail/tdk-corporation/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; Through hole Manufacturing Part Number (none) -> FG14X7R1H334KNT06
- Q101, Q102: Through Hole Digikey (none) -> https://www.digikey.com/en/products/detail/onsemi/2N7000/24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; Through hole Manufacturing Part Number (none) -> 2N7000
- R101, R102, R103, R104, R106, R108: Through Hole Digikey (none) -> https://www.digikey.com/en/products/detail/stackpole-electr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; Through hole Manufacturing Part Number (none) -> CF12JT4K70
- R105: Through Hole Digikey (none) -> https://www.digikey.com/en/products/detail/te-connectivity-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; Through hole Manufacturing Part Number (none) -> ROX1SJ15K
- R107, R110: Through Hole Digikey (none) -> https://www.digikey.com/en/products/detail/vishay-dale/CPF1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; Through hole Manufacturing Part Number (none) -> CPF1100K00FKEE6
- R109: Through Hole Digikey (none) -> https://www.digikey.com/en/products/detail/stackpole-electr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; Through hole Manufacturing Part Number (none) -> CF14JT10K0
- U101, U105, U106: Through Hole Digikey (none) -> Connector Not Needed; Through hole Manufacturing Part Number (none) -> Connector Not Needed
- U102: Through Hole Digikey (none) -> https://www.digikey.com/en/products/detail/texas-instrument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; Through hole Manufacturing Part Number (none) -> LM555CN/NOPB
- U103: Through Hole Digikey (none) -> https://www.digikey.com/en/products/detail/vishay-semicondu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; Through hole Manufacturing Part Number (none) -> SFH617A-1
- U104: Through Hole Digikey (none) -> https://www.digikey.com/en/products/detail/texas-instrument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; Through hole Manufacturing Part Number (none) -> SN74AHC02N
- U107: Through Hole Digikey (none) -> https://www.digikey.com/en/products/detail/recom-power/RI-1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; Through hole Manufacturing Part Number (none) -> RI-1205S
