File: Fault Latch/Fault Latch 2/Through Hole Fault Latch For Physical Testing/Fault Latch 2- THT.kicad_sch (KiCad schematic)
At the start: 110 parts, among them K101 Fujitsu_FTR-LYAA005x, K102 Fujitsu_FTR-LYAA005x, K103 Fujitsu_FTR-LYAA005x, Q101 Q_NPN_BEC, Q102 Q_NPN_BEC, Q103 Q_NPN_BEC, Q104 Q_NPN_BEC, Q105 Q_NMOS_GSD, Q106 Q_NMOS_GSD, Q107 Q_PMOS_GSD, Q108 Q_PMOS_GSD, Q109 Q_PMOS_GSD, Q110 Q_NPN_BEC, Q111 Q_NPN_BEC, Q112 Q_NMOS_GSD, Q113 Q_PMOS_GSD, Q114 Q_NMOS_GSD, Q115 Q_NMOS_GSD, SW101 SW_Omron_B3FS, SW102 SW_Omron_B3FS, SW103 SW_Omron_B3FS, U101 SFH617A-1, U102 SFH617A-1, U103 SFH617A-1, U104 74AHC1G00, U105 74AHC1G00, U106 74AHC1G00, U107 74LS279, U108 641964-1, U109 SFH617A-1, U110 SFH617A-1, U111 641964-1, U112 641964-1, U113 641964-1, U114 641964-1, U115 641964-1, U116 641964-1, U117 74AHC1G00, U118 LM555xM, U119 74AHC1G00, U120 641964-1, U121 SFH617A-1, U122 641964-1, U123 641964-1

Commit message: Creating a flashlight cuz im amazing
Parts:
- C101, C105, C106, C109: Through Hole Key (none) -> https://www.digikey.com/en/products/detail/vishay-beyschlag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; Through Hole Manufacturer (none) -> A103K15X7RF5TAA
- C102, C103, C104, C108, C110, C112, C116, C117: Through Hole Key (none) -> https://www.digikey.com/en/products/detail/vishay-beyschlag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; Through Hole Manufacturer (none) -> K104K10X7RF5UH5
- C107, C114: Through Hole Key (none) -> https://www.digikey.com/en/products/detail/vishay-beyschlag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; Through Hole Manufacturer (none) -> K105K20X7RF5TH5
- C111: Through Hole Key (none) -> https://www.digikey.com/en/products/detail/tdk-corporation/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; Through Hole Manufacturer (none) -> FK14X5R0J226MR020
- C113: Through Hole Key (none) -> https://www.digikey.com/en/products/detail/tdk-corporation/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; Through Hole Manufacturer (none) -> FK20X5R0J476MN000
- C115: Through Hole Key (none) -> https://www.digikey.com/en/products/detail/tdk-corporation/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; Through Hole Manufacturer (none) -> FG14X7R1H334KNT06
- D1, D2: Through Hole Key (none) -> https://www.digikey.com/en/products/detail/stmicroelectroni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; Through Hole Manufacturer (none) -> 1N5819RL
- D101, D102, D103: Through Hole Key (none) -> https://www.digikey.com/en/products/detail/w%C3%BCrth-elekt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; Through Hole Manufacturer (none) -> 151051RS11000
- D104, D105, D106: Through Hole Key (none) -> https://www.digikey.com/en/products/detail/stmicroelectroni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; Through Hole Manufacturer (none) -> 1N5819
- H101, H102, H103, H104: Through Hole Key (none) -> https://www.digikey.com/en/products/detail/kyocera-avx/0092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; Through Hole Manufacturer (none) -> 009296001202906
- K101, K102, K103: Through Hole Key (none) -> https://www.digikey.com/en/products/detail/finder-relays-in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; Through Hole Manufacturer (none) -> 34.51.7.060.0010
- PS101: Through Hole Key (none) -> https://www.digikey.com/en/products/detail/recom-power/RD-0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; Through Hole Manufacturer (none) -> RD-0505D
- Q101, Q102, Q103, Q104, Q110, Q111: Through Hole Key (none) -> https://www.digikey.com/en/products/detail/onsemi/BC33740BU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; Through Hole Manufacturer (none) -> BC33740BU
- Q105, Q106, Q112, Q114, Q115: Through Hole Key (none) -> https://www.digikey.com/en/products/detail/infineon-technol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; Through Hole Manufacturer (none) -> IRFZ34NPBF
- Q107, Q108, Q109, Q113: Through Hole Key (none) -> https://www.digikey.com/en/products/detail/renesas-electron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; Through Hole Manufacturer (none) -> N0604N-S19-AY
- R101, R110, R113, R119, R122, R127, R132: Through Hole Key (none) -> https://www.digikey.com/en/products/detail/stackpole-electr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; Through Hole Manufacturer (none) -> CF18JT100K
- R102, R103, R104, R105, R114, R121, R123, R125, R126, R133, R134, R136: Through Hole Key (none) -> https://www.digikey.com/en/products/detail/stackpole-electr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; Through Hole Manufacturer (none) -> CF14JT10K0
- R106, R107, R108, R109, R111, R115, R120, R124, R129: Through Hole Key (none) -> https://www.digikey.com/en/products/detail/stackpole-electr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; Through Hole Manufacturer (none) -> CF14JT1K00
- R112, R135: Through Hole Key (none) -> https://www.digikey.com/en/products/detail/stackpole-electr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; Through Hole Manufacturer (none) -> CF14JT510R
- R116, R117, R118: Through Hole Key (none) -> https://www.digikey.com/en/products/detail/stackpole-electr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; Through Hole Manufacturer (none) -> CF12JT2K00
- R130: Through Hole Key (none) -> https://www.digikey.com/en/products/detail/stackpole-electr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; Through Hole Manufacturer (none) -> CF18JT270R
- R131: Through Hole Key (none) -> https://www.digikey.com/en/products/detail/stackpole-electr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; Through Hole Manufacturer (none) -> CF12JT15K0
- SW101, SW102, SW103: Through Hole Key (none) -> https://www.digikey.com/en/products/detail/omron-electronic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; Through Hole Manufacturer (none) -> B3FS-1000
- U101, U102, U103, U109, U110, U121: Through Hole Key (none) -> https://www.digikey.com/en/products/detail/liteon/LTV-816S/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; Through Hole Manufacturer (none) -> LTV-816S
- U104, U105, U106, U117, U119: Through Hole Key (none) -> https://www.digikey.com/en/products/detail/texas-instrument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; Through Hole Manufacturer (none) -> SN74LV1T00DCKR
- U107: Through Hole Key (none) -> https://www.digikey.com/en/products/detail/nexperia-usa-inc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; Through Hole Manufacturer (none) -> HEF4043BT,653
- U108, U111, U112, U113, U114, U115, U116, U120, U122, U123: Through Hole Key (none) -> https://www.digikey.com/en/products/detail/te-connectivity-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; Through Hole Manufacturer (none) -> 641964-1
- U118: Through Hole Key (none) -> https://www.digikey.com/en/products/detail/texas-instrument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; Through Hole Manufacturer (none) -> LM555CMX/NOPB
