File: Projects/Sang N./flashlight/flashlight.kicad_sch (KiCad schematic)
At the start: 0 parts

Commit message: added flashlight
Parts:
- added D1: LED, symbol Device:LED
- added R2: R, symbol Device:R
- added SW2: SW_SPST, symbol Switch:SW_SPST

Commit message: Revert "added flashlight"
This reverts commit 114a32e43cf8345afc968644d8f8c5cfb0c2f7a2.
Parts:
- removed D1: LED, symbol Device:LED
- removed R2: R, symbol Device:R
- removed SW2: SW_SPST, symbol Switch:SW_SPST
