File: Projects/Luka Brekalo/Flashilight/Flashilight.kicad_sch (KiCad schematic)
At the start: 1 part

Commit message: hmm
Parts:
- added R1: 1k, Resistor_THT:R_Axial_DIN0207_L6.3mm_D2.5mm_P7.62mm_Horizontal, symbol Device:R_US
- added SW1: SW_Push, Button_Switch_THT:SW_TH_Tactile_Omron_B3F-10xx, symbol Switch:SW_Push
Connections:
- net at D1.1 (K): now also SW1.1
- net at D1.2 (A): now also R1.2
- new net +5V: R1.1
- new net GND: SW1.2
Other:
- moved on the sheet: D1
