File: BSPD/BSPD-revamp/BPSD-2025/SPICE/BPSD-2025.kicad_pcb (KiCad board)
At the start: 2 copper layers, 90.2 x 67 mm, 68 parts, among them J1 SAMMY-3PIN, J2 SAMMY-3PIN, J3 SAMMY-2PIN, J4 SAMMY-5PIN, J5 SAMMY-2PIN, Q1 NMOS, Q2 NMOS, U10 LM397, U11 SN74AHC1G08DBVR, U12 LM397, U17 SN74AHC1G32DBVR, U18 SN74AHC1G32DBVR, U3 LM1117DT-5.0, U4 LM397, U5 LM397, U6 LM397, U7 SN74AHC1G08DBVR, U8 SN74AHC1G00DBVR, U9 LM397

Commit message: Yianni BSPD eFuse
Parts:
- removed the ? at (101.0, 69.0)
- removed C1: 1nf, Capacitor_SMD:C_1206_3216Metric
- removed C5: 10uF, Capacitor_SMD:C_1206_3216Metric
- removed R1: 470k, Resistor_SMD:R_1210_3225Metric
- removed R2: 19.1k, Resistor_SMD:R_1210_3225Metric
- removed R3: 54.9k, Resistor_SMD:R_1206_3216Metric
- removed R4: 39k, Resistor_SMD:R_1210_3225Metric
- removed U1: ~, Package_SO:SOIC-8_3.9x4.9mm_P1.27mm
- moved C4 17.3 mm to (118.4, 85.9)
- moved TP9 2.99 mm to (101.9, 70.4)
- moved TP8 2.79 mm to (101.9, 74.4)
- moved TP10 2.20 mm to (101.9, 78.4)
Connections:
- C4 pad 1: Net-(U1-OUT) -> +12V
- U3 pad 3: Net-(U1-OUT) -> +12V
Routing:
- net Net-(U1-OUT): track 18.4 -> 0.00 mm, vias 2 -> 0
- net Net-(U1-OVP): track 15.4 -> 0.00 mm
- net Net-(U1-ENUV): track 10.2 -> 0.00 mm
- net Net-(U1-SS): track 7.02 -> 0.00 mm
- net Net-(U1-ILM): track 4.84 -> 0.00 mm
- net +12V: track 79.1 -> 83.6 mm, vias 6 -> 4
- net /THRESH_BSE: track 71.2 -> 75.2 mm, vias 5 -> 3
- net GND: track 18.4 -> 18.7 mm, vias 721 -> 777
Other:
- board text removed: "BSPD"
