File: BSPD/BSPD-revamp/BPSD-2025/SPICE/BPSD-2025.kicad_sch (KiCad schematic)
At the start: 63 parts, among them J1 SAMMY-3PIN, J2 SAMMY-3PIN, J3 SAMMY-2PIN, J4 SAMMY-5PIN, J5 SAMMY-2PIN, Q1 NMOS, Q2 NMOS, U10 LM397, U11 SN74AHC1G08DBVR, U12 LM397, U17 SN74AHC1G32DBVR, U18 SN74AHC1G32DBVR, U3 LM1117DT-5.0, U4 LM397, U5 LM397, U6 LM397, U7 SN74AHC1G08DBVR, U8 SN74AHC1G00DBVR, U9 LM397

Commit message: Yianni BSPD eFuse
Parts:
- removed C1: 1nf, Capacitor_SMD:C_1206_3216Metric, symbol Device:C
- removed C5: 10uF, Capacitor_SMD:C_1206_3216Metric, symbol Device:C
- removed R1: 470k, Resistor_SMD:R_1210_3225Metric, symbol Device:R_US
- removed R2: 19.1k, Resistor_SMD:R_1210_3225Metric, symbol Device:R_US
- removed R3: 54.9k, Resistor_SMD:R_1206_3216Metric, symbol Device:R_US
- removed R4: 39k, Resistor_SMD:R_1210_3225Metric, symbol Device:R_US
- removed U1: ~, Package_SO:SOIC-8_3.9x4.9mm_P1.27mm, symbol BSPD:TPS25921ADR
- removed U3: LM1117DT-5.0, Package_TO_SOT_SMD:TO-252-3_TabPin2, symbol Regulator_Linear:LM1117DT-5.0
- added V1: 12, symbol Simulation_SPICE:VDC
- added V2: 5, symbol Simulation_SPICE:VDC
Connections:
- net +12V: now also C4.1, V1.1
- net +5V: now also V2.1
- net GND: now also V1.2, V2.2
- no-connect marks 4 -> 3
Other:
- note removed: "about 400mA trip current"
- moved on the sheet: C2, C4, R22, R23, RV6, RV7, TP10, TP8, TP9
