File: Discharge_PCB/Discharge_PCB.kicad_pcb (KiCad board)
At the start: 2 copper layers, 7 parts, among them K1 Relay_SPST-NC, Q1 PMOS

Commit message: added data sheet for resistor
yianni make footprint for 3k
Parts:
- moved TP3 101.4 mm to (120.0, 100.0)
- moved TP2 84.7 mm to (134.0, 52.5)
- moved TP5 44.6 mm to (187.5, 50.0)
- moved TP4 28.3 mm to (201.0, 100.5)
Routing:
- net Net-(Q1-G): track 85.3 -> 13.2 mm
- net Net-(K1-Pad11): track 0.00 -> 36.1 mm
- net Net-(K1-Pad12): track 0.00 -> 36.1 mm
Changed lines of the file:
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@@
 			(psa4output no)
 			(plot_black_and_white yes)
-			(plotinvisibletext no)
 			(sketchpadsonfab no)
 			(plotpadnumbers no)
@@
 	(footprint "TestPoint:TestPoint_Loop_D2.50mm_Drill1.85mm"
 		(layer "F.Cu")
-		(at 217.5 66.65)
+		(at 134 52.5)
 		(descr "wire loop as test point, loop diameter 2.5mm, hole diameter 1.85mm")
 		(tags "test point wire loop bead")
@@
 	(footprint "TestPoint:TestPoint_Loop_D2.50mm_Drill1.85mm"
 		(layer "F.Cu")
-		(at 217.5 83)
+		(at 187.5 50)
 		(descr "wire loop as test point, loop diameter 2.5mm, hole diameter 1.85mm")
 		(tags "test point wire loop bead")
@@
 	(footprint "TestPoint:TestPoint_Loop_D2.50mm_Drill1.85mm"
 		(layer "F.Cu")
-		(at 217.5 77.55)
+		(at 201 100.5)
 		(descr "wire loop as test point, loop diameter 2.5mm, hole diameter 1.85mm")
 		(tags "test point wire loop bead")
@@
 	(footprint "TestPoint:TestPoint_Loop_D2.50mm_Drill1.85mm"
 		(layer "F.Cu")
-		(at 217.5 72.1)
+		(at 120 100)
 		(descr "wire loop as test point, loop diameter 2.5mm, hole diameter 1.85mm")
 		(tags "test point wire loop bead")
@@
 	)
 	(segment
+		(start 151.5 48.5)
+		(end 146.5 48.5)
+		(width 0.2)
+		(layer "F.Cu")
+		(net 2)
+	)
+	(segment
+		(start 146.5 49.5)
+		(end 146.46 49.54)
+		(width 0.2)
+		(layer "F.Cu")
+		(net 2)
+	)
+	(segment
+		(start 146.5 48.5)
+		(end 146.5 49.5)
+		(width 0.2)
+		(layer "F.Cu")
+		(net 2)
+	)
+	(segment
+		(start 155.5 52.5)
+		(end 151.5 48.5)
+		(width 0.2)
+		(layer "F.Cu")
+		(net 2)
+	)
+	(segment
 		(start 130.22 67.09)
 		(end 120.2 77.11)
 		(width 0.2)
 		(layer "F.Cu")
-		(net 2)
+		(net 4)
+	)
+	(segment
+		(start 120.2 77.11)
+		(end 120.2 99)
+		(width 0.2)
+		(layer "F.Cu")
+		(net 4)
 	)
 	(segment
@@
 		(width 0.2)
 		(layer "F.Cu")
-		(net 2)
-	)
-	(segment
-		(start 151.5 48.5)
-		(end 146.5 48.5)
-		(width 0.2)
-		(layer "F.Cu")
-		(net 2)
+		(net 5)
 	)
 	(segment
@@
 		(width 0.2)
 		(layer "F.Cu")
-		(net 2)
-	)
-	(segment
-		(start 146.5 49.5)
-		(end 146.46 49.54)
-		(width 0.2)
-		(layer "F.Cu")
-		(net 2)
-	)
-	(segment
-		(start 120.2 77.11)
-		(end 120.2 99)
-		(width 0.2)
-		(layer "F.Cu")
-		(net 2)
-	)
-	(segment
-		(start 146.5 48.5)
-		(end 146.5 49.5)
-		(width 0.2)
-		(layer "F.Cu")
-		(net 2)
-	)
-	(segment
-		(start 155.5 52.5)
-		(end 151.5 48.5)
-		(width 0.2)
-		(layer "F.Cu")
-		(net 2)
+		(net 5)
 	)
 	(zone
