File: Discharge_PCB/Discharge_PCB.kicad_sch (KiCad schematic)
At the start: 7 parts, among them K1 Relay_SPST-NC, Q1 PMOS

Commit message: added data sheet for resistor
yianni make footprint for 3k
Parts:
- added R1: 3k, symbol Device:R_US
Connections:
- net at K1.12: now also R1.1; no longer TP4.1
- new net: R1.2, TP4.1
Other:
- moved on the sheet: TP4, TP5
Changed lines of the file:
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@@
 	(wire
 		(pts
-			(xy 176.53 87.63) (xy 176.53 92.71)
-		)
-		(stroke
-			(width 0)
-			(type default)
-		)
-	)
-	(wire
-		(pts
-			(xy 152.4 95.25) (xy 161.29 95.25)
-		)
-		(stroke
-			(width 0)
-			(type default)
-		)
-	)
-	(wire
-		(pts
-			(xy 152.4 87.63) (xy 176.53 87.63)
+			(xy 152.4 95.25) (xy 157.48 95.25)
+		)
+		(stroke
+			(width 0)
+			(type default)
+		)
+	)
+	(wire
+		(pts
+			(xy 152.4 87.63) (xy 193.04 87.63)
+		)
+		(stroke
+			(width 0)
+			(type default)
+		)
+	)
+	(wire
+		(pts
+			(xy 193.04 87.63) (xy 193.04 96.52)
 		)
 		(stroke
@@
 		(pts
 			(xy 115.57 87.63) (xy 123.19 87.63)
+		)
+		(stroke
+			(width 0)
+			(type default)
+		)
+	)
+	(wire
+		(pts
+			(xy 165.1 95.25) (xy 171.45 95.25)
 		)
 		(stroke
@@
 				(path "/2e316d8b-a221-419f-b549-d02adc4cca38"
 					(reference "Q1")
+					(unit 1)
+				)
+			)
+		)
+	)
+	(symbol
+		(lib_id "Device:R_US")
+		(at 161.29 95.25 90)
+		(unit 1)
+		(exclude_from_sim no)
+		(in_bom yes)
+		(on_board yes)
+		(dnp no)
+		(property "Reference" "R1"
+			(at 161.036 101.854 90)
+			(effects
+				(font
+					(size 1.27 1.27)
+				)
+			)
+		)
+		(property "Value" "3k"
+			(at 161.036 98.044 90)
+			(effects
+				(font
+					(size 1.27 1.27)
+				)
+			)
+		)
+		(property "Footprint" ""
+			(at 161.544 94.234 90)
+			(effects
+				(font
+					(size 1.27 1.27)
+				)
+				(hide yes)
+			)
+		)
+		(property "Datasheet" "https://www.digikey.com/en/products/detail/te-connectivity-passive-product/HSA503K0J/5587244?s=N4IgjCBcoEwAwA4CsVQGMoDMCGAbAzgKYA0IA9lANogDMABANYDyAFgLb4gC6pADgC5QQAVQB2AS35NMAWULZ8AVwBOhEAF91pGFRAAJAMoBBJHG7qgA"
+			(at 161.29 95.25 0)
+			(effects
+				(font
+					(size 1.27 1.27)
+				)
+				(hide yes)
+			)
+		)
+		(property "Description" "Resistor, US symbol"
+			(at 161.29 95.25 0)
+			(effects
+				(font
+					(size 1.27 1.27)
+				)
+				(hide yes)
+			)
+		)
+		(pin "1"
+		)
+		(pin "2"
+		)
+		(instances
+			(project ""
+				(path "/2e316d8b-a221-419f-b549-d02adc4cca38"
+					(reference "R1")
 					(unit 1)
 				)
@@
 	(symbol
 		(lib_id "Connector:TestPoint")
-		(at 176.53 92.71 180)
+		(at 193.04 96.52 180)
 		(unit 1)
 		(exclude_from_sim no)
@@
 		(dnp no)
 		(property "Reference" "TP5"
-			(at 180.848 96.012 90)
+			(at 197.358 99.822 90)
 			(effects
 				(font
@@
 		)
 		(property "Value" "-12V"
-			(at 178.816 96.266 90)
+			(at 195.326 100.076 90)
 			(effects
 				(font
@@
 		)
 		(property "Footprint" "TestPoint:TestPoint_Loop_D1.80mm_Drill1.0mm_Beaded"
-			(at 171.45 92.71 0)
+			(at 187.96 96.52 0)
 			(effects
 				(font
@@
 		)
 		(property "Datasheet" "~"
-			(at 171.45 92.71 0)
+			(at 187.96 96.52 0)
 			(effects
 				(font
@@
 		)
 		(property "Description" "test point"
-			(at 176.53 92.71 0)
+			(at 193.04 96.52 0)
 			(effects
 				(font
@@
 	(symbol
 		(lib_id "Connector:TestPoint")
-		(at 161.29 95.25 270)
+		(at 171.45 95.25 270)
 		(unit 1)
 		(exclude_from_sim no)
@@
 		(dnp no)
 		(property "Reference" "TP4"
-			(at 164.592 90.932 90)
+			(at 174.752 90.932 90)
 			(effects
 				(font
@@
 		)
 		(property "Value" "HV_Out"
-			(at 164.846 92.964 90)
+			(at 175.006 92.964 90)
 			(effects
 				(font
@@
 		)
 		(property "Footprint" "TestPoint:TestPoint_Loop_D1.80mm_Drill1.0mm_Beaded"
-			(at 161.29 100.33 0)
+			(at 171.45 100.33 0)
 			(effects
 				(font
@@
 		)
 		(property "Datasheet" "~"
-			(at 161.29 100.33 0)
+			(at 171.45 100.33 0)
 			(effects
 				(font
@@
 		)
 		(property "Description" "test point"
-			(at 161.29 95.25 0)
-			(effects
-				(font
+			(at 171.45 95.25 0)
+			(effects
+				(font
