File: BSPD/BSPD-revamp/BPSD-2025/BPSD-2025.kicad_sch (KiCad schematic)
At the start: 63 parts, among them J1 SAMMY-3PIN, J2 SAMMY-3PIN, J3 SAMMY-2PIN, J4 SAMMY-5PIN, J5 SAMMY-2PIN, Q1 NMOS, Q2 NMOS, U10 LM397, U11 SN74AHC1G08DBVR, U12 LM397, U17 SN74AHC1G32DBVR, U18 SN74AHC1G32DBVR, U3 LM1117DT-5.0, U4 LM397, U5 LM397, U6 LM397, U7 SN74AHC1G08DBVR, U8 SN74AHC1G00DBVR, U9 LM397

Commit message: BSPD schematic change & RML revamp
Parts:
- removed Q2: NMOS, Package_TO_SOT_SMD:SOT-23, symbol Simulation_SPICE:NMOS
- removed R19: 10k, Resistor_SMD:R_1210_3225Metric, symbol Device:R_US
Connections:
- net BSPD_OUT: now also Q1.1 (D)
- net GND: no longer C5.2
- new net GNDPWR: C5.2
Other:
- note added: "1"
- note added: "2"
- note added: "3"
- note added: "4"
- note added: "From 26 ESF"
- company: (none) -> TigerRacing
- title: (none) -> BSPD
- moved on the sheet: C1, C10, C11, C15, C16, C17, C18, C19, C2, C20, C21, C22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
