File: RML/RML-Yianni-Revamp/RML-Yianni-Revamp.kicad_pcb (KiCad board)
At the start: 2 copper layers, 72.6 x 32.5 mm, 45 parts, among them J1 Tractive, J3 SAMMY-6PIN, Q1 NMOS, Q2 NMOS, U1 LM397, U2 SFH617A-1, U3 LM1117DT-5.0, U4 74AHC1G02, U5 LM555xM

Commit message: Molex Microfit
Parts:
- J1: value Tractive -> MICROFIT-4PIN; footprint BSPD:SAMMY-2PIN -> RML:MICROFIT-4PIN
- R11: value 900 -> 910
- moved J1 5.49 mm to (131.6, 74.9)
- renumbered J3 to J2
Routing:
- net /TS+: track 3.66 -> 0.00 mm
