File: RML/RML-Yianni-Revamp/RML-Yianni-Revamp.kicad_sch (KiCad schematic)
At the start: 41 parts, among them J1 Tractive, J2 GLV, J3 RML1, J4 RML2, Q1 NMOS, Q2 NMOS, U1 LM397, U102 LM555xM, U104 74AHC1G02, U110 SFH617A-1, U3 LM1117DT-5.0

Commit message: RML
Parts:
- removed C101: 1u, Capacitor_SMD:C_0603_1608Metric, symbol Device:C_Polarized_US
- removed C102: 0.1u, Capacitor_SMD:C_0402_1005Metric, symbol Device:C
- removed J2: GLV, CONN_SD-105313-100_02_MOL, symbol BSPD:SAMMY-2PIN
- removed J3: RML1, CONN_SD-105313-100_02_MOL, symbol BSPD:SAMMY-2PIN
- removed J4: RML2, CONN_SD-105313-100_02_MOL, symbol BSPD:SAMMY-2PIN
- added C10: 1u, Capacitor_SMD:C_0603_1608Metric, symbol Device:C
- added C11, C12: 100n, Capacitor_SMD:C_0603_1608Metric, symbol Device:C
- added J3: SAMMY-6PIN, BSPD:SAMMY-6PIN, symbol BSPD:SAMMY-6PIN
- C1, C3, C6, C7: footprint (none) -> Capacitor_SMD:C_0603_1608Metric; JLC# (none) -> C70225
- C2, C8, C9: footprint (none) -> Capacitor_SMD:C_0603_1608Metric; JLC# (none) -> C1592
- C4: value 10n -> 10u; footprint (none) -> Capacitor_SMD:C_0603_1608Metric; JLC# (none) -> C70225
- C5: footprint (none) -> Capacitor_SMD:C_0603_1608Metric; JLC# (none) -> C1590
- D1: footprint (none) -> Diode_SMD:D_SOD-123; JLC# (none) -> C43491
- J1: footprint CONN_SD-105313-100_02_MOL -> BSPD:SAMMY-2PIN
- PS1: Digikey Link (none) -> https://www.digikey.com/en/products/detail/xp-power/IA1212D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
- Q1, Q2: footprint (none) -> Package_TO_SOT_SMD:SOT-23; JLC# (none) -> C2590
- R1, R2, R3, R4: footprint (none) -> Resistor_SMD:R_1206_3216Metric; JLC (none) -> C34578
- R10: footprint (none) -> Resistor_SMD:R_1206_3216Metric; JLC# (none) -> C17960
- R11: footprint (none) -> Resistor_SMD:R_1206_3216Metric; JLC# (none) -> C137224
- R12: footprint (none) -> Resistor_SMD:R_1206_3216Metric; JLC# (none) -> C1469
- R13: footprint (none) -> Resistor_SMD:R_1206_3216Metric; JLC# (none) -> C17927
- R14: footprint (none) -> Resistor_SMD:R_1206_3216Metric; JLC# (none) -> C25664
- R15: footprint (none) -> Resistor_SMD:R_1206_3216Metric; JLC# (none) -> C17900
- R16: renamed from R109; footprint Capacitor_SMD:C_0402_1005Metric -> Resistor_SMD:R_1206_3216Metric; JLC# C102759 -> C1489
- R17: renamed from R110; footprint Capacitor_SMD:C_0402_1005Metric -> Resistor_SMD:R_1206_3216Metric; JLC# C102750 -> C17900
- R5: footprint (none) -> Resistor_SMD:R_1206_3216Metric; JLC# (none) -> C18017
- R6: footprint (none) -> Resistor_SMD:R_1206_3216Metric; JLC# (none) -> C17948
- R7, R8: footprint (none) -> Resistor_SMD:R_1206_3216Metric; JLC# (none) -> C17901
- R9: footprint (none) -> Resistor_SMD:R_1206_3216Metric; JLC# (none) -> C17986
- U1: JLC# (none) -> C132076
- U3: JLC# (none) -> C354068
- renumbered U110 to U2, U104 to U4, U102 to U5
Connections:
- net +12V: now also J3.2, J3.4, J3.6
- net +5V: now also C10.1, C11.1, C12.2
- net GND: now also C10.2, C11.2, C12.1, J3.5
- net Vref: now also R8.1; no longer R8.2
- net RML2-: now reaches Q2.1 (D)
- net RML2-: now also J3.1
- net at C4.2, U1.1 (-): now also R8.2; no longer R8.1
- net RML1-: now reaches Q1.1 (D)
- net RML1-: now also J3.3
- no-connect marks 2 -> 3

Commit message: RML BOM
Parts:
- R11: value 900 -> 910
Changed lines of the file:
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@@
 			)
 		)
-		(property "Value" "900"
+		(property "Value" "910"
 			(at 63.5 168.91 90)
 			(effects

Commit message: Molex Microfit
Parts:
- removed J1: Tractive, BSPD:SAMMY-2PIN, symbol BSPD:SAMMY-2PIN
- added J1: MICROFIT-4PIN, RML:MICROFIT-4PIN, symbol RML:MICROFIT-4PIN
- renumbered J3 to J2
Connections:
- net GNDPWR: now also J1.1
- net TS+: now also J1.2
- no-connect marks 3 -> 5
Changed lines of the file:
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@@
 	)
 	(junction
-		(at 39.37 30.48)
+		(at 48.26 30.48)
 		(diameter 0)
 		(color 0 0 0 0)
@@
 	)
 	(no_connect
+		(at 45.72 22.86)
+	)
+	(no_connect
+		(at 45.72 25.4)
+	)
+	(no_connect
 		(at 135.89 31.75)
 	)
@@
 	(wire
 		(pts
-			(xy 36.83 30.48) (xy 39.37 30.48)
+			(xy 45.72 30.48) (xy 48.26 30.48)
 		)
 		(stroke
@@
 	(wire
 		(pts
-			(xy 36.83 27.94) (xy 45.72 27.94)
+			(xy 45.72 27.94) (xy 54.61 27.94)
 		)
 		(stroke
@@
 	(wire
 		(pts
-			(xy 39.37 30.48) (xy 45.72 30.48)
+			(xy 48.26 30.48) (xy 54.61 30.48)
 		)
 		(stroke
@@
 	)
 	(label "TS+"
-		(at 45.72 27.94 180)
+		(at 54.61 27.94 180)
 		(effects
 			(font
@@
 	)
 	(label "TS-"
-		(at 45.72 30.48 180)
+		(at 54.61 30.48 180)
 		(effects
 			(font
@@
 		(dnp no)
 		(fields_autoplaced yes)
-		(property "Reference" "J3"
+		(property "Reference" "J2"
 			(at 26.67 35.56 0)
 			(effects
@@
 			(project ""
 				(path "/6fc260e6-9c33-4f6e-9221-b841b900d5e4"
-					(reference "J3")
+					(reference "J2")
 					(unit 1)
 				)
@@
 	)
 	(symbol
-		(lib_id "BSPD:SAMMY-2PIN")
-		(at 36.83 30.48 180)
-		(unit 1)
-		(exclude_from_sim no)
-		(in_bom yes)
-		(on_board yes)
-		(dnp no)
-		(fields_autoplaced yes)
-		(property "Reference" "J1"
-			(at 27.94 20.32 0)
-			(effects
-				(font
-					(size 1.524 1.524)
-				)
-			)
-		)
-		(property "Value" "Tractive"
-			(at 27.94 22.86 0)
-			(effects
-				(font
-					(size 1.524 1.524)
-				)
-			)
-		)
-		(property "Footprint" "BSPD:SAMMY-2PIN"
-			(at 28.448 24.13 0)
-			(effects
-				(font
-					(size 1.27 1.27)
-					(italic yes)
-				)
-				(hide yes)
-			)
-		)
-		(property "Datasheet" "https://www.molex.com/en-us/products/part-detail-pdf/1053131202?display=pdf"
-			(at 24.384 21.336 0)
-			(effects
-				(font
-					(size 1.27 1.27)
-					(italic yes)
-				)
-				(hide yes)
-			)
-		)
-		(property "Description" ""
-			(at 36.83 30.48 0)
-			(effects
-				(font
-					(size 1.27 1.27)
-				)
-				(hide yes)
-			)
-		)
-		(pin "2"
-		)
-		(pin "1"
-		)
-		(instances
-			(project ""
-				(path "/6fc260e6-9c33-4f6e-9221-b841b900d5e4"
-					(reference "J1")
-					(unit 1)
-				)
-			)
-		)
-	)
-	(symbol
 		(lib_id "Device:R_US")
 		(at 134.62 107.95 0)
@@
 	(symbol
 		(lib_id "power:GNDPWR")
-		(at 39.37 30.48 0)
+		(at 48.26 30.48 0)
 		(unit 1)
 		(exclude_from_sim no)
@@
 		(fields_autoplaced yes)
 		(property "Reference" "#PWR01"
-			(at 39.37 35.56 0)
+			(at 48.26 35.56 0)
 			(effects
 				(font
@@
 		)
 		(property "Value" "GNDPWR"
-			(at 39.243 34.29 0)
+			(at 48.133 34.29 0)
 			(effects
 				(font
@@
 		)
 		(property "Footprint" ""
-			(at 39.37 31.75 0)
+			(at 48.26 31.75 0)
 			(effects
 				(font
@@
 		)
 		(property "Datasheet" ""
-			(at 39.37 31.75 0)
+			(at 48.26 31.75 0)
 			(effects
 				(font
@@
 		)
 		(property "Description" "Power symbol creates a global label with name \"GNDPWR\" , global ground"
-			(at 39.37 30.48 0)
+			(at 48.26 30.48 0)
 			(effects
 				(font
@@
 					(unit 1)
 				)
+			)
+		)
+	)
+	(symbol
+		(lib_id "RML:MICROFIT-4PIN")
+		(at 45.72 30.48 180)
+		(unit 1)
+		(exclude_from_sim no)
+		(in_bom yes)
+		(on_board yes)
+		(dnp no)
+		(property "Reference" "J1"
+			(at 40.386 16.002 0)
+			(effects
+				(font
+					(size 1.524 1.524)
+				)
+			)
+		)
+		(property "Value" "MICROFIT-4PIN"
+			(at 40.386 18.542 0)
+			(effects
+				(font
+					(size 1.524 1.524)
+				)
+			)
+		)
+		(property "Footprint" "RML:MICROFIT-4PIN"
+			(at 45.72 30.48 0)
+			(effects
+				(font
+					(size 1.27 1.27)
+					(italic yes)
+				)
+				(hide yes)
+			)
+		)
+		(property "Datasheet" "https://www.molex.com/en-us/products/part-detail-pdf/447640401?display=pdf"
+			(at 45.72 30.48 0)
+			(effects
+				(font
+					(size 1.27 1.27)
+					(italic yes)
+				)
+				(hide yes)
+			)
+		)
+		(property "Description" ""
+			(at 45.72 30.48 0)
+			(effects
+				(font
+					(size 1.27 1.27)
+				)
+				(hide yes)
+			)
+		)
+		(pin "1"
+		)
+		(pin "3"
+		)
+		(pin "4"
+		)
+		(pin "2"
+		)
+		(instances
+			(project ""
+				(path "/6fc260e6-9c33-4f6e-9221-b841b900d5e4"
+					(reference "J1")
+					(unit 1)
+				)
