File: TS_Schematics/TS_Schematic26/TS_Schematic26.kicad_sch (KiCad schematic)
At the start: 1 part, among them U1 TRACTIVE

Commit message: Updated TS Schematics 4 esf
esf dtuff
Parts:
- added K1: Discharge_NC, symbol Relay:Relay_SPST-NC
- added R1, R2: 10K, symbol Device:R_US
- added R3: 3K, symbol Device:R_US
- added U2: ~, symbol TS:HVIL
- added U3: ~, symbol TS:HV_500
- added U4: ~, symbol TS:EMRAX_208_HV
- added U5: ~, symbol TS:Energy_Meter
- added U6: ~, symbol TS:MSD
- U1: value TRACTIVE -> TRACTIVE SYSTEM BATTERY
Connections:
- net 1 AWG: now reaches U1. (3)
- net 1 AWG: now also K1.11, R3.1, U2., U3. (Phase_3), U5. (OUT), U6.
- new net: K1.12, R3.2
- new net: U3. (Phase_3), U4. (Phase_3) (x3)
- new net GND: K1.A1
- new net Shudown Signal: K1.A2
- new net TSMP+: R1.1
- new net TSMP-: R2.2
Other:
- added sheet Tractive Battery Schematic (untitled.kicad_sch)
- note added: "HVIL"
- note added: "MINIMSDF000R"
- moved on the sheet: U1
