File: Fault Latch/Fault Latch 2/Fault Latch 2.kicad_sch (KiCad schematic)
At the start: 104 parts, among them J1 1053141312, J3 1053131202, J4 1053131202, K3 Fujitsu_FTR-LYCA005x, K5 Fujitsu_FTR-LYCA005x, K6 Fujitsu_FTR-LYCA005x, Q101 Q_NPN_BEC, Q102 Q_NPN_BEC, Q103 Q_NPN_BEC, Q104 Q_NPN_BEC, Q105 Q_NMOS_GSD, Q106 Q_NMOS_GSD, Q110 Q_NPN_BEC, Q111 Q_NPN_BEC, Q112 Q_NMOS_GSD, Q113 Q_NMOS_GSD, Q114 Q_NMOS_GSD, Q115 Q_NMOS_GSD, Q117 Q_NMOS_GSD, Q118 Q_NMOS_GSD, Q120 Q_NMOS_GSD, SW101 SW_Omron_B3FS, SW102 SW_Omron_B3FS, SW103 SW_Omron_B3FS, U1 74LS279, U101 SFH617A-1, U104 74AHC1G00, U108 SFH617A-1, U109 74AHC1G00, U111 SFH617A-1, U112 74AHC1G00, U117 74AHC1G00, U118 LM555xM, U2 LM1117DT-5.0, U7 SN74AHC1G08DBVR, U8 SN74AHC1G08DBVR

Commit message: Changed Optocoupler to mosfet and added resistor to tssi red
Parts:
- removed R102, R125: 220, Resistor_SMD:R_0805_2012Metric_Pad1.20x1.40mm_HandSolder, symbol Device:R_US
- removed U101, U108, U111: SFH617A-1, Package_DIP:DIP-4_W7.62mm, symbol Isolator:SFH617A-1
- added Q119, Q121, Q122: Q_NMOS_GSD, Package_TO_SOT_SMD:SOT-23, symbol Transistor_FET:Q_NMOS_GSD
- added R138, R139, R140: 10k, Resistor_SMD:R_0805_2012Metric_Pad1.20x1.40mm_HandSolder, symbol Device:R_US
- R133: value 220 -> 680; footprint Resistor_SMD:R_0805_2012Metric_Pad1.20x1.40mm_HandSolder -> Resistor_SMD:R_0805_2012Metric; JLC# C17557 -> C1359; Manufacturer_Part_Number (none) -> CR0805-JW-681ELF
Connections:
- net +12V: no longer R133.2
- net BSPD_HV: now also Q122.1 (G), R140.1
- net GND: now also Q119.2 (S), Q121.2 (S), Q122.2 (S), R138.2, R139.2, R140.2
- net IMD_HV: now also Q121.1 (G), R139.1
- net NBMS_HV: now also Q119.1 (G), R138.1
- net NBMS_LV: now also Q119.3 (D)
- net NBPSD_LV: now also Q122.3 (D)
- net NIMD_LV: now also Q121.3 (D)
- net at U7.4: now also R133.2; no longer Q113.1 (G)
- net at R133.1: now also Q113.1 (G)
Other:
- note added: "BMS Wiring Manual"

Commit message: Fault Latch V3
Parts:
- added J5: 1053131202, Connector_Molex:Molex_Nano-Fit_105313-xx02_1x02_P2.50mm_Horizontal, symbol molex.2-pin:1053131202
- added Q123, Q124, Q125: Q_NMOS_GSD, Package_TO_SOT_SMD:SOT-23, symbol Transistor_FET:Q_NMOS_GSD
- added R107, R109, R116: 1k, Resistor_SMD:R_0805_2012Metric_Pad1.20x1.40mm_HandSolder, symbol Device:R_US
- added U3: ~, Package_TO_SOT_SMD:SOT-223, symbol New_Library:BTS4141NHUMA1_
Connections:
- net +12V: now also R107.1, R109.1, R116.1, U3.1 (OUT); no longer J3.2
- net BSPD_HV: now also Q125.1 (G); no longer Q122.1 (G)
- net GND: now also Q123.2 (S), Q124.2 (S), Q125.2 (S)
- net IMD_HV: now also Q124.1 (G); no longer Q121.1 (G)
- net NBMS_HV: now also Q123.1 (G); no longer Q119.1 (G)
- new net: Q122.1 (G), Q125.3 (D), R116.2
- new net: Q119.1 (G), Q123.3 (D), R107.2
- new net: Q121.1 (G), Q124.3 (D), R109.2
- new net LVB: J3.2, U3.4 (V_BB)
- new net Load Switch +: J5.1, U3.3 (IN)
- new net Load Switch -: J5.2, U3.2 (GND)
Other:
- moved on the sheet: C101, C102, C105, C106, C107, C108, C109, C110, C111, C112, C113, C114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
